Commit message: feat: complete refactor of robot description with modular xacro and launch files

File: urdf/my_robot.urdf.xacro (robot description, xacro)
@@ -3,3 +3,23 @@
   <xacro:include filename="robot_core.xacro"/>
   <xacro:robot_core/>
+  <ros2_control name="MyRobot" type="system">
+    <hardware>
+      <plugin>mock_components/GenericSystem</plugin>
+    </hardware>
+    <joint name="shoulder_joint">
+      <command_interface name="position"/>
+      <state_interface name="position"/>
+      <state_interface name="velocity"/>
+    </joint>
+    <joint name="elbow_link_joint">
+      <command_interface name="position"/>
+      <state_interface name="position"/>
+      <state_interface name="velocity"/>
+    </joint>
+    <joint name="wrist_joint">
+      <command_interface name="position"/>
+      <state_interface name="position"/>
+      <state_interface name="velocity"/>
+    </joint>
+  </ros2_control>
 </robot>

File: urdf/robot_core.xacro (robot description, xacro)
@@ -1,101 +1,80 @@
+<?xml version="1.0"?>
 <robot xmlns:xacro="http://www.ros.org/wiki/xacro">
-<xacro:macro name="robot_core">
-<xacro:property name="chassis_size" value="1 1 1"/>
-<xacro:property name="shoulder_len" value="0.3"/>
-<xacro:property name="elbow_len" value="0.4"/>
-<xacro:property name="wrist_offset" value="0.25"/>
-<xacro:macro name="arm_segment" params="name parent length radius origin_z axis">
-    <link name="${name}">
-        <visual>
-            <geometry>
-                <cylinder length="${length}" radius="${radius}"/>
-            </geometry>
-        </visual>
-    </link>
-    <joint name="${name}_joint" type="revolute">
-        <parent link="${parent}"/>
-        <child link="${name}"/>
-        <origin xyz="0 0 ${origin_z}"/>
-        <axis xyz="${axis}"/>
-        <limit lower="-3.14" upper="3.14" effort="10" velocity="1"/>
-    </joint>
-</xacro:macro>
-<link name="base_link"></link>
-<link name ="chassis_link">
-    <visual>
+  <xacro:macro name="robot_core">
+    <!-- ================= BASE ================= -->
+    <link name="base_link"/>
+    <link name="chassis_link">
+      <visual>
         <geometry>
-            <box size="${chassis_size}"/>
+          <box size="1 1 1"/>
         </geometry>
         <material name="red">
-            <color rgba="1 0 0 1"/>
+          <color rgba="1 0 0 1"/>
         </material>
-    </visual>
-    <collision>
+      </visual>
+    </link>
+    <joint name="base_to_chassis" type="fixed">
+      <parent link="base_link"/>
+      <child link="chassis_link"/>
+      <origin xyz="0 0 0.5"/>
+    </joint>
+    <!-- ================= SHOULDER ================= -->
+    <link name="shoulder">
+      <visual>
+        <origin xyz="0 0 0.15"/>
         <geometry>
-            <box size="1 1 1"/>
+          <cylinder length="0.3" radius="0.1"/>
         </geometry>
-    </collision>
-</link>
-<xacro:arm_segment
-    name="shoulder_link"
-    parent="chassis_link"
-    length="${shoulder_len}"
-    radius="0.1"
-    origin_z="0.5"
-    axis="0 0 1"/>
-<xacro:arm_segment
-    name="elbow_link"
-    parent="shoulder_link"
-    length="${elbow_len}"
-    radius="0.08"
-    origin_z="${shoulder_len}"
-    axis="0 0 1"/>
-<link name="wrist_link">
-    <visual>
+      </visual>
+    </link>
+    <joint name="shoulder_joint" type="revolute">
+      <parent link="chassis_link"/>
+      <child link="shoulder"/>
+      <origin xyz="0 0 0.5"/>
+      <axis xyz="0 0 1"/>
+      <limit lower="-3.14" upper="3.14" effort="10" velocity="1"/>
+    </joint>
+    <!-- ================= ELBOW ================= -->
+    <link name="elbow_link">
+      <visual>
+        <origin xyz="0 0 0.2"/>
         <geometry>
-            <box size="0.75 0.5 0.5"/>
+          <cylinder length="0.4" radius="0.08"/>
+        </geometry>
+      </visual>
+    </link>
+    <joint name="elbow_link_joint" type="revolute">
+      <parent link="shoulder"/>
+      <child link="elbow_link"/>
+      <origin xyz="0 0 0.3"/>
+      <axis xyz="0 0 1"/>
+      <limit lower="-3.14" upper="3.14" effort="10" velocity="1"/>
+    </joint>
+    <!-- ================= WRIST ================= -->
+    <link name="wrist_link">
+      <visual>
+        <origin xyz="0 0 0.2"/>
+        <geometry>
+          <box size="0.4 0.4 0.4"/>
         </geometry>
         <material name="blue">
-            <color rgba="0 0 1 1"/>
+          <color rgba="0 0 1 1"/>
         </material>
-    </visual>
-    <collision>
+      </visual>
+      <collision>
+        <origin xyz="0 0 0.2"/>
         <geometry>
-            <box size="0.75 0.5 0.5"/>
+          <box size="0.4 0.4 0.4"/>
         </geometry>
-    </collision>
-    <inertial>
-    <mass value="0.25"/>
-    <origin xyz="0 0 0"/>
-        <inertia
-            ixx="0.1" ixy="0.0" ixz="0.0"
-            iyy="0.1" iyz="0.0"
-            izz="0.1"/>
-    </inertial>
-</link>
-<link name="camera_link">
-    <visual>
-        <geometry>
-            <box size="0.2 0.2 0.2"/>
-        </geometry>
-    </visual>
-</link>
-<joint name="base_to_chassis" type="fixed">
-    <parent link="base_link"/>
-    <child link="chassis_link"/>
-    <origin xyz="0 0 0.5" rpy="0 0 0"/>
-</joint>
-<joint name="wrist_joint" type="revolute">
-    <parent link="elbow_link"/>
-    <child link="wrist_link"/>
-    <origin xyz="0 0 ${elbow_len}"/>
-    <axis xyz="1 0 0"/>
-    <limit lower="-1.57" upper="1.57" effort="10" velocity="1"/>
-</joint>
-<joint name="camera_joint" type="fixed">
-    <parent link="wrist_link"/>
-    <child link="camera_link"/>
-    <origin xyz="0 0 ${wrist_offset}"/>
-</joint>
-</xacro:macro>
+      </collision>
+    </link>
+    <joint name="wrist_joint" type="revolute">
+      <parent link="elbow_link"/>
+      <child link="wrist_link"/>
+      <!-- 🔥 FIX: NO VARIABLE -->
+      <origin xyz="0 0 0.4"/>
+      <axis xyz="1 0 0"/>
+      <limit lower="-1.57" upper="1.57" effort="10" velocity="1"/>
+    </joint>
+  </xacro:macro>
 </robot>
