Commit message: feat: add inertial and collision tags to robot_core for physics simulation

File: urdf/robot_core.xacro (robot description, xacro)
@@ -3,5 +3,11 @@
   <xacro:macro name="robot_core">
     <!-- ================= BASE ================= -->
-    <link name="base_link"/>
+    <link name="base_link">
+      <collision>
+        <geometry>
+          <box size="0.1 0.1 0.1"/>
+        </geometry>
+      </collision>
+    </link>
     <link name="chassis_link">
       <visual>
@@ -13,4 +19,17 @@
         </material>
       </visual>
+      <collision>
+        <geometry>
+          <box size="1 1 1"/>
+        </geometry>
+      </collision>
+      <inertial>
+        <mass value="2.0"/>
+        <origin xyz="0 0 0"/>
+        <inertia
+          ixx="0.1" ixy="0.0" ixz="0.0"
+          iyy="0.1" iyz="0.0"
+          izz="0.1"/>
+      </inertial>
     </link>
     <joint name="base_to_chassis" type="fixed">
@@ -27,4 +46,18 @@
         </geometry>
       </visual>
+      <collision>
+        <origin xyz="0 0 0.15"/>
+        <geometry>
+          <cylinder length="0.3" radius="0.1"/>
+        </geometry>
+      </collision>
+      <inertial>
+        <mass value="1.0"/>
+        <origin xyz="0 0 0.15"/>
+        <inertia
+          ixx="0.01" ixy="0.0" ixz="0.0"
+          iyy="0.01" iyz="0.0"
+          izz="0.01"/>
+      </inertial>
     </link>
     <joint name="shoulder_joint" type="revolute">
@@ -43,4 +76,18 @@
         </geometry>
       </visual>
+      <collision>
+        <origin xyz="0 0 0.2"/>
+        <geometry>
+          <cylinder length="0.4" radius="0.08"/>
+        </geometry>
+      </collision>
+      <inertial>
+        <mass value="0.5"/>
+        <origin xyz="0 0 0.2"/>
+        <inertia
+          ixx="0.01" ixy="0.0" ixz="0.0"
+          iyy="0.01" iyz="0.0"
+          izz="0.01"/>
+      </inertial>
     </link>
     <joint name="elbow_link_joint" type="revolute">
@@ -68,9 +115,16 @@
         </geometry>
       </collision>
+      <inertial>
+        <mass value="0.5"/>
+        <origin xyz="0 0 0.2"/>
+        <inertia
+          ixx="0.01" ixy="0.0" ixz="0.0"
+          iyy="0.01" iyz="0.0"
+          izz="0.01"/>
+      </inertial>
     </link>
     <joint name="wrist_joint" type="revolute">
       <parent link="elbow_link"/>
       <child link="wrist_link"/>
-      <!-- 🔥 FIX: NO VARIABLE -->
       <origin xyz="0 0 0.4"/>
       <axis xyz="1 0 0"/>
